Commit message: Adapt driver for ROS 2 Lyrical and Gazebo simulation

File: staubli_robot_description/r2c/staubli.r2c.xacro (robot description, xacro)
@@ -12,4 +12,5 @@
         initial_positions_file:=^
         use_mock_hardware:=^
+        use_gazebo_hardware:=false
         mock_sensor_commands:=^
     ">
@@ -19,31 +20,55 @@
     <ros2_control name="${name}" type="system">
         <hardware>
-            <xacro:if value="${use_mock_hardware}">
-                <plugin>mock_components/GenericSystem</plugin>
-                <param name="calculate_dynamics">true</param>
-                <param name="state_following_offset">0.0</param>
-                <param name="mock_sensor_commands">${mock_sensor_commands}</param>
+            <!-- Selección del plugin de hardware.
+                 - use_gazebo_hardware=true  -> gz_ros2_control (simulación Gazebo Sim).
+                   Se usa `gz_ros2_control/GazeboSimSystem` porque es el plugin que
+                   Hace de puente entre el estado/comandos de las articulaciones
+                   de ros2_control y el motor de física de Gazebo Sim dentro del proceso de gz-sim.
+                 - use_mock_hardware=true    -> mock_components/GenericSystem (sin hardware).
+                 - ambos false               -> staubli_robot_driver/StaubliHardwareInterface
+                   (robot real CS9, comunicado por UDP).
+                 El default es no-Gazebo (use_gazebo_hardware=false) para no alterar el
+                 comportamiento actual de mock y hardware real. -->
+            <xacro:if value="${use_gazebo_hardware}">
+                <plugin>gz_ros2_control/GazeboSimSystem</plugin>
             </xacro:if>
-            <xacro:unless value="${use_mock_hardware}">
-                <plugin>staubli_robot_driver/StaubliHardwareInterface</plugin>
-                <param name="robot_prefix">${robot_prefix}</param>
-                <param name="robot_ip">${robot_ip}</param>
-                <param name="control_port">11000</param>
-                <param name="diagnostic_port">11001</param>
-                <param name="local_control_port">11000</param>
-                <param name="local_diagnostic_port">11001</param>
-                <param name="num_digital_inputs">${num_digital_inputs}</param>
-                <param name="num_digital_outputs">${num_digital_outputs}</param>
-                <param name="num_analog_inputs">${num_analog_inputs}</param>
-                <param name="num_analog_outputs">${num_analog_outputs}</param>
+            <xacro:unless value="${use_gazebo_hardware}">
+                <xacro:if value="${use_mock_hardware}">
+                    <plugin>mock_components/GenericSystem</plugin>
+                    <param name="calculate_dynamics">true</param>
+                    <param name="state_following_offset">0.0</param>
+                    <param name="mock_sensor_commands">${mock_sensor_commands}</param>
+                </xacro:if>
+                <xacro:unless value="${use_mock_hardware}">
+                    <plugin>staubli_robot_driver/StaubliHardwareInterface</plugin>
+                    <param name="robot_prefix">${robot_prefix}</param>
+                    <param name="robot_ip">${robot_ip}</param>
+                    <param name="control_port">11000</param>
+                    <param name="diagnostic_port">11001</param>
+                    <param name="local_control_port">11000</param>
+                    <param name="local_diagnostic_port">11001</param>
+                    <param name="num_digital_inputs">${num_digital_inputs}</param>
+                    <param name="num_digital_outputs">${num_digital_outputs}</param>
+                    <param name="num_analog_inputs">${num_analog_inputs}</param>
+                    <param name="num_analog_outputs">${num_analog_outputs}</param>
+                </xacro:unless>
             </xacro:unless>
         </hardware>
         <!-- Actuated joints -->
-        <xacro:if value="${use_mock_hardware}">
+        <!-- El comando de aceleración solo existe en el hardware real:
+             se usa únicamente para definir los límites de aceleración.
+             En mock y en Gazebo Sim (GazeboSimSystem) no se usa, porque
+             GazeboSimSystem no expone interfaz de comando `acceleration`. -->
+        <xacro:if value="${use_gazebo_hardware}">
             <xacro:property name="include_acceleration_command" value="false"/>
         </xacro:if>
-        <xacro:unless value="${use_mock_hardware}">
-             <!-- Note: acceleration command interface is ONLY used to set the acceleration limits... -->
-            <xacro:property name="include_acceleration_command" value="true"/>
+        <xacro:unless value="${use_gazebo_hardware}">
+            <xacro:if value="${use_mock_hardware}">
+                <xacro:property name="include_acceleration_command" value="false"/>
+            </xacro:if>
+            <xacro:unless value="${use_mock_hardware}">
+                 <!-- Note: acceleration command interface is ONLY used to set the acceleration limits... -->
+                <xacro:property name="include_acceleration_command" value="true"/>
+            </xacro:unless>
         </xacro:unless>
         <xacro:r2c_joints_control_description
@@ -56,26 +81,31 @@
         />
         <!-- Virtual GPIOs for Control / Supervision -->
-        <gpio name="${robot_prefix}supervision">
-            <!-- Integers -->
-            <state_interface name="operation_mode"/>
-            <state_interface name="operation_mode_status"/>
-            <state_interface name="safety_status"/>
-            <state_interface name="control_sequence_delay"/>
-            <!-- Booleans -->
-            <state_interface name="brakes_released"/>
-            <state_interface name="motion_possible"/>
-            <state_interface name="in_motion"/>
-            <state_interface name="in_error"/>
-            <state_interface name="estop_pressed"/>
-            <state_interface name="wait_for_ack"/>
-        </gpio>
-        <!-- GPIOs -->
-        <xacro:r2c_gpios_control_description
-            robot_prefix="${robot_prefix}"
-            num_digital_inputs="${num_digital_inputs}"
-            num_digital_outputs="${num_digital_outputs}"
-            num_analog_inputs="${num_analog_inputs}"
-            num_analog_outputs="${num_analog_outputs}"
-        />
+        <!-- GazeboSimSystem no soporta interfaces GPIO (digitales/analógicas), por lo que
+             los bloques <gpio> se excluyen cuando se usa Gazebo Sim. Esto no afecta al
+             robot real ni al mock hardware. -->
+        <xacro:unless value="${use_gazebo_hardware}">
+            <gpio name="${robot_prefix}supervision">
+                <!-- Integers -->
+                <state_interface name="operation_mode"/>
+                <state_interface name="operation_mode_status"/>
+                <state_interface name="safety_status"/>
+                <state_interface name="control_sequence_delay"/>
+                <!-- Booleans -->
+                <state_interface name="brakes_released"/>
+                <state_interface name="motion_possible"/>
+                <state_interface name="in_motion"/>
+                <state_interface name="in_error"/>
+                <state_interface name="estop_pressed"/>
+                <state_interface name="wait_for_ack"/>
+            </gpio>
+            <!-- GPIOs -->
+            <xacro:r2c_gpios_control_description
+                robot_prefix="${robot_prefix}"
+                num_digital_inputs="${num_digital_inputs}"
+                num_digital_outputs="${num_digital_outputs}"
+                num_analog_inputs="${num_analog_inputs}"
+                num_analog_outputs="${num_analog_outputs}"
+            />
+        </xacro:unless>
     </ros2_control>
     </xacro:macro>

File: staubli_robot_description/urdf/staubli.urdf.xacro (robot description, xacro)
@@ -33,4 +33,11 @@
     <xacro:arg name="use_mock_hardware" default="true"/>
     <xacro:arg name="mock_sensor_commands" default="false"/>
+    <!-- Path (absolute) to the controllers YAML used by gz_ros2_control.
+         Computed by launch_gazebo.launch.py y pasado como arg. -->
+    <xacro:arg name="gazebo_controllers_file" default=""/>
+    <!-- Gazebo Sim: cuando use_gazebo_hardware:=true, se usa gz_ros2_control
+         en lugar del driver real o mock. Default false para mantener el
+         comportamiento actual sin necesidad de cambiar ningún launch. -->
+    <xacro:arg name="use_gazebo_hardware" default="false"/>
     <!-- Toggle absolute / relative mesh paths -->
     <xacro:arg name="force_abs_paths" default="false"/>
@@ -68,5 +75,23 @@
         initial_positions_file="$(arg initial_positions_file)"
         use_mock_hardware="$(arg use_mock_hardware)"
+        use_gazebo_hardware="$(arg use_gazebo_hardware)"
         mock_sensor_commands="$(arg mock_sensor_commands)"
     />
+    <!-- Gazebo Sim plugin de gz_ros2_control.
+         Solo se añade cuando use_gazebo_hardware:=true. El tag <gazebo> es el
+         que soporta sdformat en la conversion URDF→SDF: se convierte en un
+         <plugin> a nivel de <model> en el SDF resultante. El nombre de la
+         clase coincide con la registrada por GZ_ADD_PLUGIN en la libreria
+         gz_ros2_control v3.0.8 (Lyrical). <parameters> es obligatorio: el
+         plugin aborta la inicializacion si esta vacio. -->
+    <xacro:if value="$(arg use_gazebo_hardware)">
+        <gazebo>
+            <plugin
+                filename="libgz_ros2_control-system.so"
+                name="gz_ros2_control::GazeboSimROS2ControlPlugin">
+                <parameters>$(arg gazebo_controllers_file)</parameters>
+                <position_proportional_gain>1.0</position_proportional_gain>
+            </plugin>
+        </gazebo>
+    </xacro:if>
 </robot>
