Commit message: Add camera laser marker visualization

File: staubli_robot_description/urdf/include/staubli_camera.xacro (robot description, xacro)
@@ -28,4 +28,7 @@
         height:=480
         hfov:=1.0472
+        laser_distance:='0.50'
+        laser_width:='0.30'
+        laser_line_width:='0.008'
     ">
         <!-- Camera mount link (eye-in-hand) -->
@@ -43,4 +46,41 @@
                 <material name="camera_material">
                     <color rgba="0.15 0.15 0.15 1"/>
+                </material>
+            </visual>
+            <visual name="camera_housing_visual">
+                <geometry>
+                    <box size="0.06 0.05 0.045"/>
+                </geometry>
+                <material name="camera_housing_material">
+                    <color rgba="0.08 0.10 0.12 1"/>
+                </material>
+            </visual>
+            <visual name="camera_lens_visual">
+                <origin xyz="0.032 0 0" rpy="0 1.57079632679 0"/>
+                <geometry>
+                    <cylinder radius="0.016" length="0.008"/>
+                </geometry>
+                <material name="camera_lens_material">
+                    <color rgba="0.02 0.04 0.08 1"/>
+                </material>
+            </visual>
+            <visual name="laser_triangle_visual">
+                <origin xyz="0 0 0" rpy="0 0 0"/>
+                <geometry>
+                    <mesh
+                        filename="package://staubli_robot_description/meshes/laser_triangle.obj"
+                        scale="${laser_distance} ${laser_width} 1.0"/>
+                </geometry>
+                <material name="laser_triangle_material">
+                    <color rgba="0.10 0.70 1.0 0.25"/>
+                </material>
+            </visual>
+            <visual name="laser_line_visual">
+                <origin xyz="${laser_distance} 0 0" rpy="0 0 0"/>
+                <geometry>
+                    <box size="${laser_line_width} ${laser_width} ${laser_line_width}"/>
+                </geometry>
+                <material name="laser_line_material">
+                    <color rgba="1.0 0.0 0.0 0.95"/>
                 </material>
             </visual>

File: staubli_robot_description/urdf/staubli.urdf.xacro (robot description, xacro)
@@ -13,4 +13,7 @@
     <xacro:arg name="robot_prefix" default=""/>
     <xacro:arg name="robot_ip" default="0.0.0.0"/>
+    <xacro:arg name="laser_distance" default="0.50"/>
+    <xacro:arg name="laser_width" default="0.30"/>
+    <xacro:arg name="laser_line_width" default="0.008"/>
     <!-- Set the robot name using the property -->
     <xacro:attribute name="name" value="$(arg name)" />
@@ -70,4 +73,7 @@
         robot_prefix="$(arg robot_prefix)"
         parent_link="$(arg robot_prefix)link_6"
+        laser_distance="$(arg laser_distance)"
+        laser_width="$(arg laser_width)"
+        laser_line_width="$(arg laser_line_width)"
     />
     <!-- ROS2 control description -->

Commit message: Checkpoint: sensor support correctly positioned on tool0 - gamma 0

File: staubli_robot_description/urdf/include/staubli_camera.xacro (robot description, xacro)
@@ -3,18 +3,10 @@
 <!-- |                                                                           | -->
 <!-- | Eye-in-hand camera mounted on link_6 of the TX2-60L (same Z as tool0).    | -->
+<!-- | Integrated with real support + sensor STL (SENSOR_BASE.stl).              | -->
 <!-- |                                                                           | -->
-<!-- | Orientation: in Gazebo Sim the camera optical axis is the local -Z axis.  | -->
-<!-- | At home the wrist (link_6) is world aligned, so a plain +X roll keeps the | -->
-<!-- | -Z pointing down into the robot. The fixed joint rpy (0.7031 0 0) instead | -->
-<!-- | rolls the camera so its -Z aims outward and slightly down, framing the    | -->
-<!-- | inspection table / workpiece (part_1) seen from the roof. Only the look   | -->
-<!-- | direction changes; the mount pose and tool0 are untouched.                | -->
-<!-- |                                                                           | -->
-<!-- | The camera link / fixed joint make camera_link part of the robot TF tree. | -->
-<!-- | The gazebo block (reference camera_link) embeds a Gazebo Sim camera       | -->
-<!-- | sensor: when gz-sim spawns the robot from the URDF, it is converted into  | -->
-<!-- | an SDF camera sensor on link camera_link of the model. The sensor         | -->
-<!-- | publishes the image on the Gazebo topic /camera/image_raw, which the      | -->
-<!-- | launch_gazebo.launch.py bridges to the ROS topic /camera/image_raw.       | -->
+<!-- | The STL contains the complete physical support + sensor. The virtual      | -->
+<!-- | camera geometry is removed to avoid duplication. camera_link is a frame   | -->
+<!-- | (no visual) with the sensor placed on the inclined face of the support.  | -->
+<!-- | Orientation estimation is pending validation (see comments).             | -->
 <!-- =========================================================================== -->
 <robot xmlns:xacro="http://wiki.ros.org/xacro">
@@ -22,72 +14,57 @@
         robot_prefix:=''
         parent_link
-        xyz:='0 0 0.07'
-        rpy:='2.9391 -1.3969 -2.9714'
         update_rate:=30
         width:=640
         height:=480
         hfov:=1.0472
-        laser_distance:='0.50'
-        laser_width:='0.30'
-        laser_line_width:='0.008'
     ">
-        <!-- Camera mount link (eye-in-hand) -->
+        <!-- Support + sensor physical geometry (STL) -->
+        <link name="${robot_prefix}sensor_support_link">
+            <inertial>
+                <mass value="0.5"/>
+                <inertia
+                    ixx="0.001846" ixy="0.0" ixz="0.0"
+                    iyy="0.000599" iyz="0.0" izz="0.002171"/>
+            </inertial>
+            <visual name="sensor_support_visual">
+                <geometry>
+                    <mesh
+                        filename="package://staubli_robot_description/meshes/SENSOR_BASE.stl"
+                        scale="0.001 0.001 0.001"/>
+                </geometry>
+            </visual>
+            <collision name="sensor_support_collision">
+                <geometry>
+                    <mesh
+                        filename="package://staubli_robot_description/meshes/SENSOR_BASE.stl"
+                        scale="0.001 0.001 0.001"/>
+                </geometry>
+            </collision>
+        </link>
+        <!-- Joint: tool0 -> sensor_support_link -->
+        <!-- TODO: validation pending - transformation from tool0 to support may need fine adjustment -->
+        <joint name="${robot_prefix}sensor_support_joint" type="fixed">
+            <parent link="${parent_link}"/>
+            <child link="${robot_prefix}sensor_support_link"/>
+            <origin xyz="0.016130 0.003110 0.168690" rpy="0 -1.570796 0"/>
+        </joint>
+        <!-- Camera frame (no geometry) - reference for real sensor -->
+        <!-- TODO: ESTIMATION PENDING VALIDATION
+             Position/orientation obtained from geometric analysis of STL (surface inclined).
+             Origin at center of inclined face. -Z_local(camera_link) aligned with estimated
+             observation direction (+n_patch). May require adjustment after Gazebo verification. -->
         <link name="${robot_prefix}camera_link">
             <inertial>
-                <mass value="0.05"/>
+                <mass value="0.5"/>
                 <inertia
-                    ixx="1.0e-5" ixy="0.0" ixz="0.0"
-                    iyy="1.0e-5" iyz="0.0" izz="1.0e-5"/>
+                    ixx="1.0e-6" ixy="0.0" ixz="0.0"
+                    iyy="1.0e-6" iyz="0.0" izz="1.0e-6"/>
             </inertial>
-            <visual name="camera_visual">
-                <geometry>
-                    <box size="0.04 0.04 0.04"/>
-                </geometry>
-                <material name="camera_material">
-                    <color rgba="0.15 0.15 0.15 1"/>
-                </material>
-            </visual>
-            <visual name="camera_housing_visual">
-                <geometry>
-                    <box size="0.06 0.05 0.045"/>
-                </geometry>
-                <material name="camera_housing_material">
-                    <color rgba="0.08 0.10 0.12 1"/>
-                </material>
-            </visual>
-            <visual name="camera_lens_visual">
-                <origin xyz="0.032 0 0" rpy="0 1.57079632679 0"/>
-                <geometry>
-                    <cylinder radius="0.016" length="0.008"/>
-                </geometry>
-                <material name="camera_lens_material">
-                    <color rgba="0.02 0.04 0.08 1"/>
-                </material>
-            </visual>
-            <visual name="laser_triangle_visual">
-                <origin xyz="0 0 0" rpy="0 0 0"/>
-                <geometry>
-                    <mesh
-                        filename="package://staubli_robot_description/meshes/laser_triangle.obj"
-                        scale="${laser_distance} ${laser_width} 1.0"/>
-                </geometry>
-                <material name="laser_triangle_material">
-                    <color rgba="0.10 0.70 1.0 0.25"/>
-                </material>
-            </visual>
-            <visual name="laser_line_visual">
-                <origin xyz="${laser_distance} 0 0" rpy="0 0 0"/>
-                <geometry>
-                    <box size="${laser_line_width} ${laser_width} ${laser_line_width}"/>
-                </geometry>
-                <material name="laser_line_material">
-                    <color rgba="1.0 0.0 0.0 0.95"/>
-                </material>
-            </visual>
         </link>
+        <!-- Joint: sensor_support_link -> camera_link -->
         <joint name="${robot_prefix}camera_fixed_joint" type="fixed">
-            <parent link="${parent_link}"/>
+            <parent link="${robot_prefix}sensor_support_link"/>
             <child link="${robot_prefix}camera_link"/>
-            <origin xyz="${xyz}" rpy="${rpy}"/>
+            <origin xyz="0.011764 0.129833 0.118716" rpy="0.785429 -0.775796 -3.141193"/>
         </joint>
         <!-- Gazebo Sim RGB camera sensor (simple configuration, no depth). -->

Commit message: Configure sensor support materials and FOV visualization
- Attach the sensor support to tool0 with the gamma +90 orientation
- Split SENSOR_BASE into structure, dark hardware and FOV plane meshes
- Add metallic/dark materials, a white translucent FOV plane and an opaque red edge line
- Add the original SENSOR + BASE.stl source mesh

File: staubli_robot_description/urdf/include/staubli_camera.xacro (robot description, xacro)
@@ -27,10 +27,52 @@
                     iyy="0.000599" iyz="0.0" izz="0.002171"/>
             </inertial>
-            <visual name="sensor_support_visual">
+            <!-- Visual 1: metallic structure of the support (components >= 30 mm) -->
+            <visual name="sensor_support_visual_structure">
                 <geometry>
                     <mesh
-                        filename="package://staubli_robot_description/meshes/SENSOR_BASE.stl"
+                        filename="package://staubli_robot_description/meshes/SENSOR_BASE_structure.stl"
                         scale="0.001 0.001 0.001"/>
                 </geometry>
+                <material name="sensor_support_structure_material">
+                    <color rgba="0.35 0.37 0.39 1.0"/>
+                </material>
+            </visual>
+            <!-- Visual 2: dark sensor housing + small hardware (components < 30 mm) -->
+            <visual name="sensor_support_visual_dark">
+                <geometry>
+                    <mesh
+                        filename="package://staubli_robot_description/meshes/SENSOR_BASE_dark.stl"
+                        scale="0.001 0.001 0.001"/>
+                </geometry>
+                <material name="sensor_support_dark_material">
+                    <color rgba="0.12 0.13 0.14 1.0"/>
+                </material>
+            </visual>
+            <!-- Visual 3: FOV plane of the sensor (fan extracted from SENSOR_BASE.stl,
+                 1108 triangles, identical geometry and pose: x -70.187..464.813,
+                 y -19.829..-19.819, z -411.451..440.826 mm) -->
+            <visual name="sensor_support_visual_plane">
+                <geometry>
+                    <mesh
+                        filename="package://staubli_robot_description/meshes/SENSOR_BASE_plane.stl"
+                        scale="0.001 0.001 0.001"/>
+                </geometry>
+                <material name="sensor_support_plane_material">
+                    <color rgba="1.0 1.0 1.0 0.25"/>
+                </material>
+            </visual>
+            <!-- Visual 4: red line on the far edge of the FOV plane.
+                 Same logic as the old laser_line_visual (thin box, laser_line_width
+                 thick) laid along the final edge of the plane:
+                 x = 464.813 mm, y = -19.825 mm, z -411.451..440.826 mm -->
+            <xacro:property name="laser_line_width" value="0.008"/>
+            <visual name="sensor_support_visual_line">
+                <origin xyz="0.464813 -0.019825 0.0146875" rpy="0 0 0"/>
+                <geometry>
+                    <box size="${laser_line_width} ${laser_line_width} 0.852277"/>
+                </geometry>
+                <material name="sensor_support_line_material">
+                    <color rgba="1.0 0.0 0.0 1.0"/>
+                </material>
             </visual>
             <collision name="sensor_support_collision">
@@ -47,5 +89,5 @@
             <parent link="${parent_link}"/>
             <child link="${robot_prefix}sensor_support_link"/>
-            <origin xyz="0.016130 0.003110 0.168690" rpy="0 -1.570796 0"/>
+            <origin xyz="-0.003110 0.016130 0.168690" rpy="0 -1.570796 1.570796"/>
         </joint>
         <!-- Camera frame (no geometry) - reference for real sensor -->

File: staubli_robot_description/urdf/staubli.urdf.xacro (robot description, xacro)
@@ -69,11 +69,8 @@
         <origin xyz="0 0 0" rpy="0 0 0"/>
     </xacro:staubli_robot>
-    <!-- Eye-in-hand RGB camera on link_6 (same Z as tool0). -->
+    <!-- Eye-in-hand RGB camera/sensor with real support STL attached to tool0. -->
     <xacro:staubli_camera
         robot_prefix="$(arg robot_prefix)"
-        parent_link="$(arg robot_prefix)link_6"
-        laser_distance="$(arg laser_distance)"
-        laser_width="$(arg laser_width)"
-        laser_line_width="$(arg laser_line_width)"
+        parent_link="$(arg robot_prefix)tool0"
     />
     <!-- ROS2 control description -->

Commit message: Set sensor camera pose

File: staubli_robot_description/urdf/include/staubli_camera.xacro (robot description, xacro)
@@ -108,5 +108,5 @@
             <parent link="${robot_prefix}sensor_support_link"/>
             <child link="${robot_prefix}camera_link"/>
-            <origin xyz="0.011764 0.129833 0.118716" rpy="0.785429 -0.775796 -3.141193"/>
+            <origin xyz="-0.064522 0.088917 0.014688" rpy="1.570796 0 -0.331612"/>
         </joint>
         <!-- Gazebo Sim RGB camera sensor (simple configuration, no depth). -->

Commit message: Save working scan path and inspection cell configuration

File: staubli_robot_description/urdf/include/staubli_camera.xacro (robot description, xacro)
@@ -108,5 +108,5 @@
             <parent link="${robot_prefix}sensor_support_link"/>
             <child link="${robot_prefix}camera_link"/>
-            <origin xyz="-0.064522 0.088917 0.014688" rpy="1.570796 0 -0.331612"/>
+            <origin xyz="-0.064522 0.088917 0.014688" rpy="-1.570796 0 -0.331612"/>
         </joint>
         <!-- Gazebo Sim RGB camera sensor (simple configuration, no depth). -->

Commit message: Fix sensor working distance and scan boundary alignment

File: staubli_robot_description/urdf/include/staubli_camera.xacro (robot description, xacro)
@@ -18,5 +18,31 @@
         height:=480
         hfov:=1.0472
+        working_distance:=0.325
+        working_line_width:=0.004
     ">
+        <!-- Green working-distance reference: the REAL width of the FOV fan
+             (SENSOR_BASE_plane.stl) at 'working_distance' along the boresight,
+             laid in the fan's physical plane (sensor_support_link frame).
+             Must match sensor_reference.fov_width_m() in staubli_gui. -->
+        <xacro:property name="fov_x0" value="-0.07018654"/>
+        <xacro:property name="fov_x1" value="0.46481345"/>
+        <xacro:property name="fov_zlo0" value="-0.00093088686"/>
+        <xacro:property name="fov_zhi0" value="0.03030657"/>
+        <xacro:property name="fov_zlo1" value="-0.41145084"/>
+        <xacro:property name="fov_zhi1" value="0.4408265"/>
+        <!-- Lateral offset of the FOV plane with respect to the boresight
+             (sensor_support_link +X). The STL was exported at y ~ -19.82 mm;
+             it is re-centred so the fan (and the green working reference)
+             lies on the boresight axis, which is what scan_path anchors. -->
+        <xacro:property name="fov_plane_y_raw" value="-0.0198237"/>
+        <xacro:property name="fov_plane_y" value="0.0"/>
+        <xacro:property name="fov_t"
+            value="${(working_distance - fov_x0) / (fov_x1 - fov_x0)}"/>
+        <xacro:property name="fov_zlo"
+            value="${fov_zlo0 + fov_t * (fov_zlo1 - fov_zlo0)}"/>
+        <xacro:property name="fov_zhi"
+            value="${fov_zhi0 + fov_t * (fov_zhi1 - fov_zhi0)}"/>
+        <xacro:property name="fov_width" value="${fov_zhi - fov_zlo}"/>
+        <xacro:property name="fov_zcenter" value="${(fov_zhi + fov_zlo) / 2}"/>
         <!-- Support + sensor physical geometry (STL) -->
         <link name="${robot_prefix}sensor_support_link">
@@ -53,4 +79,5 @@
                  y -19.829..-19.819, z -411.451..440.826 mm) -->
             <visual name="sensor_support_visual_plane">
+                <origin xyz="0 ${-fov_plane_y_raw} 0" rpy="0 0 0"/>
                 <geometry>
                     <mesh
@@ -65,8 +92,9 @@
                  Same logic as the old laser_line_visual (thin box, laser_line_width
                  thick) laid along the final edge of the plane:
-                 x = 464.813 mm, y = -19.825 mm, z -411.451..440.826 mm -->
+                 x = 464.813 mm, y = 0 mm (re-centred on the boresight),
+                 z -411.451..440.826 mm -->
             <xacro:property name="laser_line_width" value="0.008"/>
             <visual name="sensor_support_visual_line">
-                <origin xyz="0.464813 -0.019825 0.0146875" rpy="0 0 0"/>
+                <origin xyz="0.464813 0 0.0146875" rpy="0 0 0"/>
                 <geometry>
                     <box size="${laser_line_width} ${laser_line_width} 0.852277"/>
@@ -74,4 +102,18 @@
                 <material name="sensor_support_line_material">
                     <color rgba="1.0 0.0 0.0 1.0"/>
+                </material>
+            </visual>
+            <!-- Visual 5: GREEN working-distance reference, in the fan's own
+                 plane. It spans the real FOV width at 'working_distance' (from
+                 one fan edge to the other), so it is the 3D counterpart of the
+                 green line sensor_reference projects onto /camera/image_raw.
+                 Thin in X and Y, long along Z. -->
+            <visual name="sensor_support_visual_working_reference">
+                <origin xyz="${working_distance} ${fov_plane_y} ${fov_zcenter}" rpy="0 0 0"/>
+                <geometry>
+                    <box size="${working_line_width} ${working_line_width} ${fov_width}"/>
+                </geometry>
+                <material name="sensor_support_working_reference_material">
+                    <color rgba="0.153 0.682 0.376 1.0"/>
                 </material>
             </visual>
@@ -92,8 +134,10 @@
         </joint>
         <!-- Camera frame (no geometry) - reference for real sensor -->
-        <!-- TODO: ESTIMATION PENDING VALIDATION
-             Position/orientation obtained from geometric analysis of STL (surface inclined).
-             Origin at center of inclined face. -Z_local(camera_link) aligned with estimated
-             observation direction (+n_patch). May require adjustment after Gazebo verification. -->
+        <!-- Origin at the centre of the inclined mounting face. Orientation is
+             ALIGNED with the physical boresight (sensor_support_link +X): the
+             ~19 deg yaw misalignment (-0.331612 rad) was removed so the Gazebo
+             RGB camera (+X of camera_link) looks along the FOV fan axis. The
+             physical origin is kept unchanged. The green working-distance
+             reference lives on sensor_support_link, in the fan's plane. -->
         <link name="${robot_prefix}camera_link">
             <inertial>
@@ -104,9 +148,10 @@
             </inertial>
         </link>
-        <!-- Joint: sensor_support_link -> camera_link -->
+        <!-- Joint: sensor_support_link -> camera_link (orientation aligned to
+             the FOV boresight; origin unchanged) -->
         <joint name="${robot_prefix}camera_fixed_joint" type="fixed">
             <parent link="${robot_prefix}sensor_support_link"/>
             <child link="${robot_prefix}camera_link"/>
-            <origin xyz="-0.064522 0.088917 0.014688" rpy="-1.570796 0 -0.331612"/>
+            <origin xyz="-0.064522 0.088917 0.014688" rpy="-1.570796 0 0"/>
         </joint>
         <!-- Gazebo Sim RGB camera sensor (simple configuration, no depth). -->

File: staubli_robot_description/urdf/staubli.urdf.xacro (robot description, xacro)
@@ -16,4 +16,9 @@
     <xacro:arg name="laser_width" default="0.30"/>
     <xacro:arg name="laser_line_width" default="0.008"/>
+    <!-- Distancia óptima de trabajo (m): línea verde de referencia del sensor,
+         medida sobre el eje óptico de camera_link. Mismo valor por defecto que
+         sensor_reference.DEFAULT_WORKING_DISTANCE_M y que el "Scan distance"
+         inicial de la GUI (staubli_gui.scan_path.DEFAULT_SCAN_DISTANCE). -->
+    <xacro:arg name="working_distance" default="0.325"/>
     <!-- Set the robot name using the property -->
     <xacro:attribute name="name" value="$(arg name)" />
@@ -73,4 +78,5 @@
         robot_prefix="$(arg robot_prefix)"
         parent_link="$(arg robot_prefix)tool0"
+        working_distance="$(arg working_distance)"
     />
     <!-- ROS2 control description -->
